File: DMSMDS.brd (EAGLE design)
At the start: 25.4 x 32.8 mm, 11 parts

Commit message: v1
Parts:
- added C2: 22uF, resistor:C1206
- D1M1: value (none) -> D1M1
- D1M2: value (none) -> D1M2
- DC12V: value (none) -> 12V
- MS123: value (none) -> 123
- SM1: value (none) -> SM1
- SMD1: value (none) -> SMD1
- SMD2: value (none) -> SMD2
- moved DC12V 16.4 mm to (19.1, 8.89), turned to 0 degrees
- moved C1 15.3 mm to (20.8, 17.0)
- moved MS123 15.2 mm to (5.08, 19.1)
- moved R2 12.3 mm to (21.1, 22.1)
- moved R1 8.82 mm to (6.35, 14.0), turned to 270 degrees
- moved SM1 6.99 mm to (16.5, 8.89)
- flipped IC1 to the bottom, turned to 90 degrees
Connections:
- net N$8 renamed MSP
- removed net 3.3V: D1M1.8
- removed net A0: D1M1.2
- removed net D0: D1M1.3
- removed net D3: D1M2.5
- removed net D4: D1M2.6
- removed net D5: D1M1.4
- removed net D6: D1M1.5
- removed net D7: D1M1.6
- removed net D8: D1M1.7
- removed net RST: D1M1.1
- removed net RX: D1M2.2
- removed net TX: D1M2.1
- net 5.0V: now also C2.1
- net GND: now also C2.2
Routing:
- net 12V: track 44.9 -> 12.5 mm
- net MSP: track 21.8 -> 7.11 mm
- net EN: track 14.7 -> 2.09 mm
- net GND: track 0.00 -> 10.9 mm
- net MS1: track 9.29 -> 19.3 mm
- net MS2: track 6.22 -> 15.6 mm
- net N$4: track 10.2 -> 2.54 mm
- net N$2: track 10.1 -> 2.55 mm
- net N$1: track 10.1 -> 2.57 mm
- net N$3: track 10.1 -> 2.59 mm
- net 5.0V: track 27.3 -> 33.9 mm
- net MS3: track 6.38 -> 11.2 mm
- net D2: track 24.0 -> 21.9 mm
- net D1: track 24.7 -> 23.7 mm
- net N$10: track 3.49 -> 2.61 mm
Other:
- board text added: "12V"
- board text added: "2017-02-25"
- board text added: "MOTOR"
- board text removed: "2017-02-23"
- board text removed: "5V"
- board text removed: "A0"
- board text removed: "D2"
- board text removed: "D4"
- board text removed: "D6"
- board text removed: "D8"
- board text removed: "RX"
